Commit message: added fake distance sensors
Signed-off-by: Jakub Delicat <jakub.delicat@husarion.com>

File: rosbot_description/urdf/components/vl53lox.urdf.xacro (robot description, xacro)
@@ -4,9 +4,43 @@
   <xacro:macro name="vl53lox" params="parent xyz rpy prefix">
     <joint name="${parent}_${prefix}_range_joint" type="fixed">
-        <origin xyz="${xyz}" rpy="${rpy}" />
-        <parent link="${parent}" />
-        <child link="${prefix}_range" />
+      <origin xyz="${xyz}" rpy="${rpy}" />
+      <parent link="${parent}" />
+      <child link="${prefix}_range" />
     </joint>
     <link name="${prefix}_range" />
+    <!-- an IR sensor or a sonar are not implemented yet
+    https://github.com/gazebosim/gz-sensors/issues/19 -->
+    <xacro:if value="${simulation_engine == 'ignition-gazebo'}">
+      <gazebo reference="${prefix}_range">
+        <sensor name="${prefix}_range" type='gpu_lidar'>
+          <topic>/range/${prefix}</topic>
+          <frame_id>${prefix}_range</frame_id>
+          <ignition_frame_id>${prefix}_range</ignition_frame_id>
+          <update_rate>5.0</update_rate>
+          <ray>
+            <scan>
+              <horizontal>
+                <samples>1</samples>
+                <resolution>1</resolution>
+                <min_angle>-0.01</min_angle>
+                <max_angle>0.01</max_angle>
+              </horizontal>
+            </scan>
+            <range>
+              <min>0.01</min>
+              <max>0.90</max>
+              <resolution>0.02</resolution>
+            </range>
+            <noise>
+              <type>gaussian</type>
+              <mean>0.1</mean>
+              <stddev>0.005</stddev>
+            </noise>
+          </ray>
+          <always_on>true</always_on>
+          <visualize>false</visualize>
+        </sensor>
+      </gazebo>
+    </xacro:if>
   </xacro:macro>
 </robot>
